File: Atmega2560/MicrocontrollerPcb/MicrocontrollerPcb.sch (KiCad schematic (older format))
At the start: 38 parts, among them U1 ATmega2560-16AU

Commit message: Completed PCB Layout changed Input Connector footprint
Parts:
- removed +5V1, +5V2, +5V3, Analog1, Analog2, Analog3, Digital1, Digital2, Digital3, PWM1, PWM2, PWM3: Conn_02x01_Row_Letter_Last, Connector_PinHeader_2.54mm:PinHeader_2x01_P2.54mm_Vertical, symbol Connector_Generic:Conn_02x01_Row_Letter_Last
- added J1: Conn_02x12_Odd_Even, Connector_PinHeader_2.54mm:PinHeader_2x12_P2.54mm_Vertical, symbol Connector_Generic:Conn_02x12_Odd_Even
- 16MHz1: footprint Molex_Connector:crystal_resonator -> Crystal:Crystal_HC49-U_Vertical
- INPUT1: footprint Molex_Connector:01x02 -> Molex_Connector:input
Connections:
- net +5V: now also USBasp1.6 (Pin_6), J1.1 (Pin_1), J1.3 (Pin_3), J1.5 (Pin_5); no longer USBasp1.2 (Pin_2)
- net A1: now also U1.96 (PF1), J1.7 (Pin_7); no longer U1.97 (PF0)
- net A2: now also U1.95 (PF2), J1.9 (Pin_9); no longer U1.96 (PF1)
- net A3: now also U1.90 (PF7), J1.11 (Pin_11); no longer U1.95 (PF2)
- net D1: now also J1.17 (Pin_17)
- net D2: now also J1.15 (Pin_15)
- net D3: now also J1.13 (Pin_13)
- net Earth: now also Thrusters1.7 (Pin_7), USBasp1.4 (Pin_4), J1.10 (Pin_10), J1.12 (Pin_12), J1.14 (Pin_14), J1.16 (Pin_16), J1.18 (Pin_18), J1.2 (Pin_2), J1.20 (Pin_20), J1.22 (Pin_22), J1.24 (Pin_24), J1.4 (Pin_4), J1.6 (Pin_6), J1.8 (Pin_8); no longer Thrusters1.10 (Pin_10), USBasp1.6 (Pin_6)
- net MOSI: now also USBasp1.3 (Pin_3); no longer USBasp1.4 (Pin_4)
- net PWM1: now also J1.23 (Pin_23)
- net PWM2: now also J1.21 (Pin_21)
- net PWM3: now also J1.19 (Pin_19)
- net Reset: now also USBasp1.2 (Pin_2); no longer USBasp1.5 (Pin_5)
- net SCK: now also USBasp1.5 (Pin_5); no longer USBasp1.3 (Pin_3)
- net T6: now also Thrusters1.8 (Pin_8); no longer Thrusters1.9 (Pin_9)
- net T7: now also Thrusters1.10 (Pin_10); no longer Thrusters1.8 (Pin_8)
- net T8: now also Thrusters1.9 (Pin_9); no longer Thrusters1.7 (Pin_7)
- net at R3.2, Trigger1.1 (Pin_1): now also U1.97 (PF0); no longer U1.90 (PF7)
Other:
- moved on the sheet: R3, Trigger1
