File: Power-Board/PowerBoard.kicad_pcb (KiCad board)
At the start: 2 copper layers, 151.1 x 104.1 mm, 57 parts, among them J1 IN1, J10 probe3, J11 Battery_out, J12 Buck_out, J13 IN2, J14 Boost_out, J15 Buck_out, J2 Display, J3 Boost, J4 Buck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

Commit message: Intermediate PCB layout completed.
Parts:
- removed the REF** at (81.3, 144.8)
- removed the REF** at (81.3, 52.1)
- removed S1, S2: MDSR-7-10-25, footprint:MDSR71025
- added J16: Conn_01x02_Male, footprint:01x02, F.Cu at (84.7, 82.8)
- added J17: Conn_01x02_Male, footprint:01x02, F.Cu at (123.2, 75.3)
- added REF**: MountingHole_3.2mm_M3, MountingHole:MountingHole_3.2mm_M3, F.Cu at (80.4, 145.4)
- added REF**: MountingHole_3.2mm_M3, MountingHole:MountingHole_3.2mm_M3, F.Cu at (147.8, 145.5)
- added REF**: MountingHole_3.2mm_M3, MountingHole:MountingHole_3.2mm_M3, F.Cu at (147.4, 51.4)
- added REF**: MountingHole_3.2mm_M3, MountingHole:MountingHole_3.2mm_M3, F.Cu at (80.7, 51.5)
- J12, J14, J15, J5: footprint footprint:01x02 -> footprint:input
- J2: value Display -> Conn_02x13_Odd_Even; footprint Connector_PinHeader_2.54mm:PinHeader_2x07_P2.54mm_Vertical -> Connector_PinHeader_2.54mm:PinHeader_2x13_P2.54mm_Vertical
- J8: footprint footprint:CON_436500400_MOL -> Connector_PinHeader_2.54mm:PinHeader_1x04_P2.54mm_Vertical
- moved C3 405.2 mm to (85.0, 147.7), turned to 90 degrees
- moved U2 375.0 mm to (90.1, 147.1), turned to 270 degrees
- moved J2 371.1 mm to (100.3, 145.5), turned to 90 degrees
- moved C8 355.4 mm to (122.9, 88.3), turned to 270 degrees
- moved J8 354.9 mm to (94.5, 142.2), turned to 270 degrees
- moved U3 350.9 mm to (108.0, 74.9), turned to 270 degrees
- moved D4 350.7 mm to (105.4, 108.8), turned to 180 degrees
- moved J6 346.4 mm to (137.2, 133.3)
- moved D3 345.3 mm to (106.6, 88.7), turned to 90 degrees
- moved J7 341.9 mm to (138.8, 141.3)
- moved C6 336.4 mm to (115.9, 82.7), turned to 180 degrees
- moved J9 334.2 mm to (146.1, 125.7)
- moved J3 330.2 mm to (138.4, 68.6), turned to 90 degrees
- moved J15 329.4 mm to (148.6, 105.4), turned to 90 degrees
- moved D1 327.4 mm to (133.3, 123.2)
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Connections:
- C2 pad 1: /+5V -> /5V
- C7 pad 1: /+5V -> /5V
- CS1 pad 6: /+5V -> /5V
- CS2 pad 6: /+5V -> /5V
- J1 pad 1: Net-(J1-Pad1) -> GND
- J11 pad 1: /Battery1 -> /RV1
- J12 pad 1: /Buck_Out -> GND
- J12 pad 2: GND -> /Buck_Out
- J13 pad 2: Net-(J13-Pad2) -> GND
- J14 pad 1: /BOOST_OUT -> GND
- J14 pad 2: GND -> /BOOST_OUT
- J15 pad 1: /Buck_Out -> GND
- J15 pad 2: GND -> /Buck_Out
- J2 pad 10: /SCK -> Net-(J2-Pad10)
- J2 pad 11: /SI -> /TP_IRQ
- J2 pad 13: /K2 -> /RST
- J2 pad 14: /K3 -> GND
- J2 pad 3: GND -> Net-(J2-Pad3)
- J2 pad 4: /RST -> /5V
- J2 pad 5: /RS -> Net-(J2-Pad5)
- J2 pad 6: /TP_IRQ -> GND
- J2 pad 7: /TP_SO -> Net-(J2-Pad7)
- J2 pad 8: /TP_CS -> Net-(J2-Pad8)
- J2 pad 9: /LCD_CS -> GND
- J3 pad 1: /B1B -> /BOOST_OUT
- J3 pad 3: /BOOST_OUT -> GND
- J3 pad 4: GND -> /B1B
- J4 pad 3: /Buck_Out -> GND
- J4 pad 4: GND -> /Buck_Out
- J5 pad 1: /Buck_Out -> GND
- J5 pad 2: GND -> /Buck_Out
- Q1 pad 1: Net-(J1-Pad1) -> Net-(J1-Pad2)
- Q1 pad 2: Net-(J1-Pad1) -> Net-(J1-Pad2)
- Q1 pad 3: Net-(J1-Pad1) -> Net-(J1-Pad2)
- R4 pad 1: Net-(J1-Pad1) -> Net-(J1-Pad2)
- U1 pad 11: /RST -> /K1
- U1 pad 12: /RS -> /K2
- U1 pad 14: /TP_IRQ -> /K3
- U1 pad 15: /TP_SO -> /LCD_CS
- U1 pad 17: /LCD_CS -> /TP_SO
- U1 pad 19: /INT -> /RS
- U1 pad 20: /leak_signal -> /RST
- U1 pad 21: /CTRL1 -> /leak_signal
- U1 pad 22: /CTRL2 -> /TP_IRQ
- U1 pad 24: /K1 -> Net-(U1-Pad24)
- U1 pad 25: /K2 -> /CTRL1
- U1 pad 26: /K3 -> /CTRL2
- U1 pad 27: /TP_SO -> Net-(U1-Pad27)
- U1 pad 29: /CSB -> Net-(U1-Pad29)
- U1 pad 6: Net-(U1-Pad6) -> /INT
- U1 pad 7: Net-(U1-Pad7) -> /CSB
- U3 pad 2: /MIN1 -> /MIN2
- U3 pad 4: /MIN3 -> /MIN4
- U3 pad 7: /MIN4 -> /MIN1
- U3 pad 9: /MIN2 -> /MIN3
Routing:
- net GND: track 0.00 -> 197.0 mm, vias 0 -> 1
- net /5V: track 0.00 -> 148.8 mm, vias 0 -> 1
- net /3.3V: track 0.00 -> 116.5 mm
- net /TP_IRQ: track 0.00 -> 59.7 mm
- net /Buck_Out: track 0.00 -> 53.9 mm
- net Net-(J1-Pad2): track 0.00 -> 52.5 mm
- net /CTRL1: track 0.00 -> 50.2 mm
- net /MOUT: track 0.00 -> 43.1 mm, vias 0 -> 2
- net /CTRL2: track 0.00 -> 41.5 mm
- net /RV1: track 0.00 -> 41.4 mm
- net /SCK: track 0.00 -> 39.6 mm
- net /MIN4: track 0.00 -> 38.3 mm, vias 0 -> 2
- net /B1B: track 0.00 -> 36.1 mm
- net /RST: track 0.00 -> 36.0 mm
- net /RS: track 0.00 -> 34.4 mm
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- added copper zone on F.Cu, net /MOS1
- added copper zone on F.Cu, net /RV1
- added copper zone on B.Cu, net GND
- added copper zone on F.Cu, net Net-(J1-Pad2)
Other:
- board size 151.1 x 104.1 mm -> 76.2 x 102.9 mm

Commit message: Power Board completed
Parts:
- removed the REF** at (80.4, 145.4)
- removed the REF** at (147.8, 145.5)
- removed the REF** at (147.4, 51.4)
- removed the REF** at (80.7, 51.5)
- added J18: Battery_out, footprint:input, F.Cu at (79.0, 128.3)
- added J19: Battery_out, footprint:input, F.Cu at (78.7, 120.4)
- added J20: Battery_out, footprint:input, F.Cu at (78.7, 112.8)
- added J21: Battery_out, footprint:input, F.Cu at (79.0, 136.4)
- added J22: Conn_01x02_Male, footprint:01x02, F.Cu at (111.8, 104.1)
- added REF**: MountingHole_3.2mm_M3, MountingHole:MountingHole_3.2mm_M3, F.Cu at (80.6, 151.1)
- added REF**: MountingHole_3.2mm_M3, MountingHole:MountingHole_3.2mm_M3, F.Cu at (149.2, 150.5)
- added REF**: MountingHole_3.2mm_M3, MountingHole:MountingHole_3.2mm_M3, F.Cu at (148.6, 51.4)
- added REF**: MountingHole_3.2mm_M3, MountingHole:MountingHole_3.2mm_M3, F.Cu at (80.6, 51.4)
- moved C3 63.5 mm to (147.9, 139.0), turned to 180 degrees
- moved R7 59.4 mm to (146.3, 136.3), turned to 0 degrees
- moved U2 58.8 mm to (147.3, 133.9), turned to 0 degrees
- moved R6 54.1 mm to (145.1, 131.3), turned to 90 degrees
- moved J9 52.2 mm to (96.5, 109.2)
- moved J10 52.2 mm to (96.5, 116.8)
- moved J8 49.6 mm to (142.4, 129.5), turned to 0 degrees
- moved J7 43.3 mm to (96.5, 132.1)
- moved J6 41.6 mm to (96.5, 124.5)
- moved R11 36.2 mm to (103.5, 128.3)
- moved R10 35.6 mm to (101.6, 128.9)
- moved R13 32.4 mm to (102.2, 118.1)
- moved Q2 31.4 mm to (102.9, 123.2), turned to 90 degrees
- moved R19 29.4 mm to (107.8, 80.7), turned to 90 degrees
- moved D1 28.5 mm to (105.4, 117.5), turned to 180 degrees
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Connections:
- U1 pad 10: /SI -> /K2
- U1 pad 11: /K1 -> /K3
- U1 pad 12: /K2 -> /TP_IRQ
- U1 pad 14: /K3 -> /RST
- U1 pad 15: /LCD_CS -> /RS
- U1 pad 16: /TP_CS -> /SI
- U1 pad 19: /RS -> /SCK
- U1 pad 20: /RST -> /TP_CS
- U1 pad 21: /leak_signal -> /TX
- U1 pad 22: /TP_IRQ -> /RX
- U1 pad 24: Net-(U1-Pad24) -> /CTRL1
- U1 pad 25: /CTRL1 -> /CTRL2
- U1 pad 26: /CTRL2 -> /leak_signal
- U1 pad 29: Net-(U1-Pad29) -> /LCD_CS
- U1 pad 9: /SCK -> /K1
Routing:
- net /3.3V: track 116.5 -> 261.9 mm
- net /TP_CS: track 19.4 -> 76.6 mm
- net /K1: track 13.6 -> 68.3 mm
- net /K3: track 13.3 -> 64.3 mm
- net /K2: track 15.8 -> 65.1 mm
- net /RV1: track 41.4 -> 90.0 mm
- net /SI: track 25.9 -> 72.0 mm
- net /RS: track 34.4 -> 76.3 mm
- net /RST: track 36.0 -> 76.9 mm
- net /TP_SO: track 31.2 -> 72.1 mm
- net /SCK: track 39.6 -> 74.8 mm
- net /5V: track 148.8 -> 169.6 mm
- net /TP_IRQ: track 59.7 -> 74.8 mm
- net /MOUT: track 43.1 -> 57.1 mm, vias 2 -> 1
- net /LCD_CS: track 18.2 -> 26.3 mm
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Other:
- board size 76.2 x 102.9 mm -> 77.5 x 107.9 mm

Commit message: issue resolved
Parts:
- removed REF** (x4): MountingHole_3.2mm_M3, MountingHole:MountingHole_3.2mm_M3
- added H1: MountingHole, MountingHole:MountingHole_3.2mm_M3, F.Cu at (148.6, 51.5)
- added H2: MountingHole, MountingHole:MountingHole_3.2mm_M3, F.Cu at (80.6, 151.1)
- added H3: MountingHole, MountingHole:MountingHole_3.2mm_M3, F.Cu at (80.6, 51.4)
- added H4: MountingHole, MountingHole:MountingHole_3.2mm_M3, F.Cu at (149.3, 150.5)
Other:
- outline, holes or cut-outs redrawn
