File: Power-Board/PowerBoard.sch (KiCad schematic (older format))
At the start: 42 parts, among them J1 Conn_01x02_Male, J10 probe3, J3 Boost, J4 Buck, J6 probe1, J7 probe4, J8 bmp388, J9 probe2, Q1 IRFZ34PBF, Q2 MMBT3906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

Commit message: issues resolved
Parts:
- removed J?: Conn_01x02_Male, symbol Connector:Conn_01x02_Male
- removed Q?: IRFZ34PBF, TO254P465X1024X2050-3P, symbol SamacSys_Parts:IRFZ34PBF
- removed R? (x2): R, symbol Device:R
- added D? (x3): LED, symbol Device:LED
- added J?: B2, symbol Connector:Conn_01x02_Male
- added J?: Battery_out, symbol Connector:Conn_01x02_Male
- added J?: Boost_out, symbol Connector:Conn_01x02_Male
- added J? (x3): Buck_out, symbol Connector:Conn_01x02_Male
- added Q?: IRFZ34PBF, TO254P465X1024X2050-3P, symbol SamacSys_Parts:IRFZ34PBF
- added R2, R?: 150, symbol Device:R
- added R?: 10k, symbol Device:R
- added R?: 20k, symbol Device:R
- added R? (x3): R, symbol Device:R
- added SW? (x2): SW_Reed, symbol Switch:SW_Reed
- J1: value Conn_01x02_Male -> B1
- R1, R8: value 1k -> 2k
- R3, R9: value 5k -> 10k
- R4: value R -> 10k
- R5: value R -> 20k
- gave numbers to parts that had none: 1
Connections:
- net labels added: BOOST_OUT, Battery1, Buck_Out, INT
- net labels removed: B1, POWER, Vr
- wire segments 168 -> 176
Other:
- moved on the sheet: R4, R5

Commit message: resistance values added to LED
Parts:
- R17, R18, R19: renamed from R?; value R -> .5k
- gave numbers to parts that had none: 15
Changed lines of the file:
@@
 $EndComp
 $Comp
-L Switch:SW_Reed SW?
+L Switch:SW_Reed SW1
 U 1 1 60AD44C7
 P 2300 800
-F 0 "SW?" H 2300 1022 50  0000 C CNN
+F 0 "SW1" H 2300 1022 50  0000 C CNN
 F 1 "SW_Reed" H 2300 931 50  0000 C CNN
 F 2 "" H 2300 800 50  0001 C CNN
@@
 	2150 1650 2150 1200
 $Comp
-L SamacSys_Parts:IRFZ34PBF Q?
+L SamacSys_Parts:IRFZ34PBF Q3
 U 1 1 60B4DB43
 P 5050 1300
-F 0 "Q?" H 5479 1446 50  0000 L CNN
+F 0 "Q3" H 5479 1446 50  0000 L CNN
 F 1 "IRFZ34PBF" H 5479 1355 50  0000 L CNN
 F 2 "TO254P465X1024X2050-3P" H 5500 1250 50  0001 L CNN
@@
 MOS2
 $Comp
-L Connector:Conn_01x02_Male J?
+L Connector:Conn_01x02_Male J13
 U 1 1 60B4DB4B
 P 3850 1100
-F 0 "J?" H 3956 1278 50  0000 C CNN
+F 0 "J13" H 3956 1278 50  0000 C CNN
 F 1 "B2" H 3956 1187 50  0000 C CNN
 F 2 "" H 3850 1100 50  0001 C CNN
@@
 	4700 1100 4700 600
 $Comp
-L Device:R R?
+L Device:R R14
 U 1 1 60B4DB54
 P 4900 1200
-F 0 "R?" H 4970 1246 50  0000 L CNN
+F 0 "R14" H 4970 1246 50  0000 L CNN
 F 1 "10k" H 4970 1155 50  0000 L CNN
 F 2 "" V 4830 1200 50  0001 C CNN
@@
 $EndComp
 $Comp
-L Device:R R?
+L Device:R R15
 U 1 1 60B4DB5B
 P 4900 1500
-F 0 "R?" H 4970 1546 50  0000 L CNN
+F 0 "R15" H 4970 1546 50  0000 L CNN
 F 1 "20k" H 4970 1455 50  0000 L CNN
 F 2 "" V 4830 1500 50  0001 C CNN
@@
 	4050 1200 4750 1200
 $Comp
-L Device:R R?
+L Device:R R16
 U 1 1 60B4DB65
 P 5350 750
-F 0 "R?" H 5420 796 50  0000 L CNN
+F 0 "R16" H 5420 796 50  0000 L CNN
 F 1 "150" H 5420 705 50  0000 L CNN
 F 2 "" V 5280 750 50  0001 C CNN
@@
 $EndComp
 $Comp
-L Switch:SW_Reed SW?
+L Switch:SW_Reed SW2
 U 1 1 60B4DB6D
 P 4900 800
-F 0 "SW?" H 4900 1022 50  0000 C CNN
+F 0 "SW2" H 4900 1022 50  0000 C CNN
 F 1 "SW_Reed" H 4900 931 50  0000 C CNN
 F 2 "" H 4900 800 50  0001 C CNN
@@
 	4900 600  5350 600
 $Comp
-L Connector:Conn_01x02_Male J?
+L Connector:Conn_01x02_Male J11
 U 1 1 60B6C722
 P 3300 6900
-F 0 "J?" H 3406 7078 50  0000 C CNN
+F 0 "J11" H 3406 7078 50  0000 C CNN
 F 1 "Battery_out" H 3406 6987 50  0000 C CNN
 F 2 "" H 3300 6900 50  0001 C CNN
@@
 $EndComp
 $Comp
-L Connector:Conn_01x02_Male J?
+L Connector:Conn_01x02_Male J14
 U 1 1 60B6C7FA
 P 4050 6900
-F 0 "J?" H 4156 7078 50  0000 C CNN
+F 0 "J14" H 4156 7078 50  0000 C CNN
 F 1 "Boost_out" H 4156 6987 50  0000 C CNN
 F 2 "" H 4050 6900 50  0001 C CNN
@@
 $EndComp
 $Comp
-L Connector:Conn_01x02_Male J?
+L Connector:Conn_01x02_Male J12
 U 1 1 60B768CC
 P 3650 7350
-F 0 "J?" H 3756 7528 50  0000 C CNN
+F 0 "J12" H 3756 7528 50  0000 C CNN
 F 1 "Buck_out" H 3756 7437 50  0000 C CNN
 F 2 "" H 3650 7350 50  0001 C CNN
@@
 $EndComp
 $Comp
-L Connector:Conn_01x02_Male J?
+L Connector:Conn_01x02_Male J5
 U 1 1 60B8099F
 P 3000 7350
-F 0 "J?" H 3106 7528 50  0000 C CNN
+F 0 "J5" H 3106 7528 50  0000 C CNN
 F 1 "Buck_out" H 3106 7437 50  0000 C CNN
 F 2 "" H 3000 7350 50  0001 C CNN
@@
 	2750 7600 2750 6650
 $Comp
-L Connector:Conn_01x02_Male J?
+L Connector:Conn_01x02_Male J15
 U 1 1 60BB32BF
 P 4300 7350
-F 0 "J?" H 4406 7528 50  0000 C CNN
+F 0 "J15" H 4406 7528 50  0000 C CNN
 F 1 "Buck_out" H 4406 7437 50  0000 C CNN
 F 2 "" H 4300 7350 50  0001 C CNN
@@
 GND
 $Comp
-L Device:LED D?
+L Device:LED D4
 U 1 1 60C569AD
 P 6800 3350
-F 0 "D?" H 6792 3095 50  0000 C CNN
+F 0 "D4" H 6792 3095 50  0000 C CNN
 F 1 "LED" H 6792 3186 50  0000 C CNN
 F 2 "" H 6800 3350 50  0001 C CNN
@@
 $EndComp
 $Comp
-L Device:LED D?
+L Device:LED D3
 U 1 1 60C60B9B
 P 6800 2800
-F 0 "D?" H 6792 2545 50  0000 C CNN
+F 0 "D3" H 6792 2545 50  0000 C CNN
 F 1 "LED" H 6792 2636 50  0000 C CNN
 F 2 "" H 6800 2800 50  0001 C CNN
@@
 $EndComp
 $Comp
-L Device:LED D?
+L Device:LED D2
 U 1 1 60C6AD7A
 P 6800 2250
-F 0 "D?" H 6792 1995 50  0000 C CNN
+F 0 "D2" H 6792 1995 50  0000 C CNN
 F 1 "LED" H 6792 2086 50  0000 C CNN
 F 2 "" H 6800 2250 50  0001 C CNN
@@
 GND
 $Comp
-L Device:R R?
+L Device:R R17
 U 1 1 60C9DD1C
 P 6650 2400
-F 0 "R?" H 6720 2446 50  0000 L CNN
-F 1 "R" H 6720 2355 50  0000 L CNN
+F 0 "R17" H 6720 2446 50  0000 L CNN
+F 1 ".5k" H 6720 2355 50  0000 L CNN
 F 2 "" V 6580 2400 50  0001 C CNN
 F 3 "~" H 6650 2400 50  0001 C CNN
@@
 $EndComp
 $Comp
-L Device:R R?
+L Device:R R18
 U 1 1 60C9DDF1
 P 6650 2950
-F 0 "R?" H 6720 2996 50  0000 L CNN
-F 1 "R" H 6720 2905 50  0000 L CNN
+F 0 "R18" H 6720 2996 50  0000 L CNN
+F 1 ".5k" H 6720 2905 50  0000 L CNN
 F 2 "" V 6580 2950 50  0001 C CNN
 F 3 "~" H 6650 2950 50  0001 C CNN
@@
 $EndComp
 $Comp
-L Device:R R?
+L Device:R R19
 U 1 1 60CA7FD7
 P 6650 3500
-F 0 "R?" H 6720 3546 50  0000 L CNN
-F 1 "R" H 6720 3455 50  0000 L CNN
+F 0 "R19" H 6720 3546 50  0000 L CNN
+F 1 ".5k" H 6720 3455 50  0000 L CNN
 F 2 "" V 6580 3500 50  0001 C CNN
 F 3 "~" H 6650 3500 50  0001 C CNN

Commit message: BMP issue resolved
Connections:
- net labels added: CSB
- wire segments 176 -> 177
Changed lines of the file:
@@
 3.3V
 Text Label 4400 5650 0    50   ~ 0
-3.3V
+CSB
 Text Label 6100 6250 0    50   ~ 0
 3.3V
@@
 Wire Notes Line
 	6300 3950 6300 1900
+Wire Wire Line
+	9950 5350 10200 5350
+Text Label 10200 5350 0    50   ~ 0
+CSB
 $EndSCHEMATC

Commit message: Initiated the PCB layout."
Parts:
- removed Q1, Q3: IRFZ34PBF, TO254P465X1024X2050-3P, symbol SamacSys_Parts:IRFZ34PBF
- removed R15: 20k, symbol Device:R
- removed R16: 150, symbol Device:R
- added M1, M2: MPMOS, symbol pspice:MPMOS
- C1, C2, C3, C4, C5, C6, C7, C8: footprint (none) -> Capacitor_SMD:C_0603_1608Metric_Pad1.05x0.95mm_HandSolder
- D1, D2, D3, D4: footprint (none) -> LED_THT:LED_D3.0mm
- J1: value B1 -> IN1; footprint (none) -> battery_connector:molex_supersabre_1x2_172043-0201
- J10, J12, J14, J15, J5, J6, J7, J9: footprint (none) -> footprint:01x02
- J11: footprint (none) -> battery_connector:molex_supersabre_1x2_172043-0201
- J13: value B2 -> IN2; footprint (none) -> battery_connector:molex_supersabre_1x2_172043-0201
- J2: value Conn_02x07_Counter_Clockwise -> Display; footprint (none) -> Connector_PinHeader_2.54mm:PinHeader_2x07_P2.54mm_Vertical
- J3, J4, J8: footprint (none) -> footprint:CON_436500400_MOL
- R1, R10, R11, R12, R17, R18, R19, R3, R4, R5, R6, R7, R8, R9: footprint (none) -> Resistor_SMD:R_0603_1608Metric_Pad1.05x0.95mm_HandSolder
- R13: footprint (none) -> Resistor_SMD:R_0805_2012Metric_Pad1.15x1.40mm_HandSolder
- R14: value 10k -> 20k; footprint (none) -> Resistor_SMD:R_0603_1608Metric_Pad1.05x0.95mm_HandSolder
- R2: value 150 -> 10k; footprint (none) -> Resistor_SMD:R_0603_1608Metric_Pad1.05x0.95mm_HandSolder
- U2: symbol BMP388:BMP388 -> PowerBoard-rescue:BMP388-BMP388
Connections:
- wire segments 177 -> 184
Other:
- moved on the sheet: R4, R5

Commit message: Aiwaye
Parts:
- removed M1, M2: MPMOS, symbol pspice:MPMOS
- removed SW1, SW2: SW_Reed, symbol Switch:SW_Reed
- removed U1: Pico-MCU_RaspberryPi_and_Boards, RPi_Pico:RPi_Pico_SMD_TH, symbol PowerBoard-rescue:Pico-MCU_RaspberryPi_and_Boards
- added Q1, Q3: SIS427EDN-T1-GE3, footprint:SIS862DNT1GE3, symbol SIS427EDN-T1-GE3:SIS427EDN-T1-GE3
- added S1, S2: MDSR-7-10-25, footprint:MDSR71025, symbol MDSR-7-10-25:MDSR-7-10-25
- added U1: Pico, footprint:RPi_Pico_SMD_TH, symbol MCU_RaspberryPi_and_Boards:Pico
- CS1, CS2: footprint SOIC127P600X175-8N -> footprint:SOIC127P600X175-8N
- D1, D2, D3, D4: footprint LED_THT:LED_D3.0mm -> LED_SMD:LED_0603_1608Metric
- Q2: footprint SOT95P240X120-3N -> footprint:SOT95P240X120-3N
- U2: footprint PQFN50P200X200X80-10N -> footprint:PQFN50P200X200X80-10N
- U3: footprint DGS10_TEX -> footprint:DGS10_TEX
Connections:
- wire segments 184 -> 202

Commit message: Intermediate PCB layout completed.
Parts:
- removed J2: Display, Connector_PinHeader_2.54mm:PinHeader_2x07_P2.54mm_Vertical, symbol Connector_Generic:Conn_02x07_Counter_Clockwise
- removed S1, S2: MDSR-7-10-25, footprint:MDSR71025, symbol MDSR-7-10-25:MDSR-7-10-25
- added J16, J17: Conn_01x02_Male, footprint:01x02, symbol Connector:Conn_01x02_Male
- added J2: Conn_02x13_Odd_Even, Connector_PinHeader_2.54mm:PinHeader_2x13_P2.54mm_Vertical, symbol Connector_Generic:Conn_02x13_Odd_Even
- J12, J14, J15, J5: footprint footprint:01x02 -> footprint:input
- J8: footprint footprint:CON_436500400_MOL -> Connector_PinHeader_2.54mm:PinHeader_1x04_P2.54mm_Vertical
- U1: symbol MCU_RaspberryPi_and_Boards:Pico -> PowerBoard-rescue:Pico-MCU_RaspberryPi_and_Boards
Connections:
- net labels removed: +5V, Battery1
- wire segments 202 -> 212
Other:
- moved on the sheet: J1

Commit message: Power Board completed
Parts:
- added J18, J19, J20, J21: Battery_out, footprint:input, symbol Connector:Conn_01x02_Male
- added J22: Conn_01x02_Male, footprint:01x02, symbol Connector:Conn_01x02_Male
Connections:
- net CTRL1: now also U1.24 (GPIO18); no longer U1.25 (GPIO19)
- net CTRL2: now also U1.25 (GPIO19); no longer U1.26 (GPIO20)
- net GND: now also J18.2 (Pin_2), J19.2 (Pin_2), J20.2 (Pin_2), J21.2 (Pin_2)
- net K1: now also U1.9 (GPIO6); no longer U1.11 (GPIO8)
- net K2: now also U1.10 (GPIO7); no longer U1.12 (GPIO9)
- net K3: now also U1.11 (GPIO8); no longer U1.14 (GPIO10)
- net LCD_CS: now also U1.29 (GPIO22); no longer U1.15 (GPIO11)
- net RS: now also U1.15 (GPIO11); no longer U1.19 (GPIO14)
- net RST: now also U1.14 (GPIO10); no longer U1.20 (GPIO15)
- net RV1: now also J18.1 (Pin_1), J19.1 (Pin_1), J20.1 (Pin_1), J21.1 (Pin_1)
- net SCK: now also U1.19 (GPIO14); no longer U1.9 (GPIO6)
- net SI: now also U1.16 (GPIO12); no longer U1.10 (GPIO7)
- net TP_CS: now also U1.20 (GPIO15); no longer U1.16 (GPIO12)
- net TP_IRQ: now also U1.12 (GPIO9); no longer U1.22 (GPIO17)
- net leak_signal: now also U1.26 (GPIO20); no longer U1.21 (GPIO16)
- new net RX: J22.1 (Pin_1), U1.22 (GPIO17)
- new net TX: J22.2 (Pin_2), U1.21 (GPIO16)
Other:
- moved on the sheet: J12, J14, J15, J5
Changed lines of the file:
@@
 	9950 5150 10200 5150
 Wire Wire Line
-	10200 5750 9950 5750
-Text Label 10200 5750 0    50   ~ 0
+	10200 5850 9950 5850
+Text Label 10200 5850 0    50   ~ 0
 CTRL1
 $Comp
@@
 	8550 4650 8250 4650
 Wire Wire Line
-	8550 5050 8250 5050
-Wire Wire Line
-	8550 5150 8250 5150
+	8550 6050 8250 6050
+Wire Wire Line
+	8550 5750 8250 5750
 Text Label 5950 5350 0    50   ~ 0
 3.3V
@@
 Text Label 8250 4650 0    50   ~ 0
 SCL
-Text Label 8250 5050 0    50   ~ 0
+Text Label 8250 6050 0    50   ~ 0
 SCK
-Text Label 8250 5150 0    50   ~ 0
+Text Label 8250 5750 0    50   ~ 0
 SI
 Text Label 4450 6050 0    50   ~ 0
@@
 	2850 5500 2550 5500
 Wire Wire Line
-	10200 5650 9950 5650
+	10200 5750 9950 5750
 Text Label 2850 5500 0    50   ~ 0
 CTRL2
@@
 Text Label 650  5800 0    50   ~ 0
 MIN4
-Text Label 10200 5650 0    50   ~ 0
+Text Label 10200 5750 0    50   ~ 0
 CTRL2
 Text Label 4800 4500 0    50   ~ 0
@@
 Wire Notes Line
 	5450 7600 5450 6650
-Text Label 9950 6150 0    50   ~ 0
+Text Label 9950 5650 0    50   ~ 0
 leak_signal
 Wire Wire Line
-	9950 6150 10250 6150
-Wire Wire Line
-	8550 6150 8250 6150
-Text Label 8250 6150 0    50   ~ 0
+	9950 5650 10250 5650
+Wire Wire Line
+	8550 5550 8250 5550
+Text Label 8250 5550 0    50   ~ 0
 RST
-Text Label 8250 6050 0    50   ~ 0
+Text Label 8250 5650 0    50   ~ 0
 RS
 Wire Wire Line
-	8250 6050 8550 6050
+	8250 5650 8550 5650
 Wire Wire Line
 	8250 5450 8550 5450
@@
 TP_SO
 Wire Wire Line
-	8300 5250 8550 5250
+	8300 5050 8550 5050
 Wire Wire Line
 	9700 5750 9950 5750
-Text Label 8300 5250 0    50   ~ 0
+Text Label 8300 5050 0    50   ~ 0
 K1
-Text Label 8250 5350 0    50   ~ 0
+Text Label 8250 5150 0    50   ~ 0
 K2
-Text Label 8250 5550 0    50   ~ 0
+Text Label 8250 5250 0    50   ~ 0
 K3
 Wire Wire Line
@@
 Text Label 2050 7650 0    50   ~ 0
 TP_CS
-Text Label 10250 6050 0    50   ~ 0
+Text Label 8250 5350 0    50   ~ 0
 TP_IRQ
 Text Label 8250 5850 0    50   ~ 0
 TP_SO
-Text Label 8250 5750 0    50   ~ 0
+Text Label 8300 6150 0    50   ~ 0
 TP_CS
-Text Label 8250 5650 0    50   ~ 0
+Text Label 9950 5350 0    50   ~ 0
 LCD_CS
 Wire Wire Line
-	9950 6050 10250 6050
+	8250 5350 8550 5350
 Wire Wire Line
 	8250 5850 8550 5850
 Wire Wire Line
-	8250 5750 8550 5750
-Wire Wire Line
-	8250 5650 8550 5650
+	8300 6150 8550 6150
+Wire Wire Line
+	9950 5350 10250 5350
 Connection ~ 3950 2900
 Wire Wire Line
@@
 L Connector:Conn_01x02_Male J14
 U 1 1 60B6C7FA
-P 4050 6900
-F 0 "J14" H 4156 7078 50  0000 C CNN
-F 1 "Boost_out" H 4156 6987 50  0000 C CNN
-F 2 "footprint:input" H 4050 6900 50  0001 C CNN
-F 3 "~" H 4050 6900 50  0001 C CNN
-	1    4050 6900
+P 3950 7250
+F 0 "J14" H 4056 7428 50  0000 C CNN
+F 1 "Boost_out" H 4056 7337 50  0000 C CNN
+F 2 "footprint:input" H 3950 7250 50  0001 C CNN
+F 3 "~" H 3950 7250 50  0001 C CNN
+	1    3950 7250
 	1    0    0    -1
 $EndComp
@@
 L Connector:Conn_01x02_Male J12
 U 1 1 60B768CC
-P 3650 7350
-F 0 "J12" H 3756 7528 50  0000 C CNN
-F 1 "Buck_out" H 3756 7437 50  0000 C CNN
-F 2 "footprint:input" H 3650 7350 50  0001 C CNN
-F 3 "~" H 3650 7350 50  0001 C CNN
-	1    3650 7350
+P 3100 7300
+F 0 "J12" H 3206 7478 50  0000 C CNN
+F 1 "Buck_out" H 3206 7387 50  0000 C CNN
+F 2 "footprint:input" H 3100 7300 50  0001 C CNN
+F 3 "~" H 3100 7300 50  0001 C CNN
+	1    3100 7300
 	1    0    0    -1
 $EndComp
@@
 L Connector:Conn_01x02_Male J5
 U 1 1 60B8099F
-P 3000 7350
-F 0 "J5" H 3106 7528 50  0000 C CNN
-F 1 "Buck_out" H 3106 7437 50  0000 C CNN
-F 2 "footprint:input" H 3000 7350 50  0001 C CNN
-F 3 "~" H 3000 7350 50  0001 C CNN
-	1    3000 7350
+P 2800 7300
+F 0 "J5" H 2906 7478 50  0000 C CNN
+F 1 "Buck_out" H 2906 7387 50  0000 C CNN
+F 2 "footprint:input" H 2800 7300 50  0001 C CNN
+F 3 "~" H 2800 7300 50  0001 C CNN
+	1    2800 7300
 	1    0    0    -1
 $EndComp
@@
 L Connector:Conn_01x02_Male J15
 U 1 1 60BB32BF
-P 4300 7350
-F 0 "J15" H 4406 7528 50  0000 C CNN
-F 1 "Buck_out" H 4406 7437 50  0000 C CNN
-F 2 "footprint:input" H 4300 7350 50  0001 C CNN
-F 3 "~" H 4300 7350 50  0001 C CNN
-	1    4300 7350
+P 3500 7250
+F 0 "J15" H 3606 7428 50  0000 C CNN
+F 1 "Buck_out" H 3606 7337 50  0000 C CNN
+F 2 "footprint:input" H 3500 7250 50  0001 C CNN
+F 3 "~" H 3500 7250 50  0001 C CNN
+	1    3500 7250
 	1    0    0    -1
 $EndComp
@@
 Wire Notes Line
 	2750 7600 4700 7600
-Text Label 4250 7000 0    50   ~ 0
+Text Label 4150 7350 0    50   ~ 0
 BOOST_OUT
 Text Label 3500 6900 0    50   ~ 0
@@
 Text Label 3500 7000 0    50   ~ 0
 GND
-Text Label 4250 6900 0    50   ~ 0
+Text Label 4150 7250 0    50   ~ 0
 GND
 $Comp
@@
 	1    0    0    -1
 $EndComp
-Text Label 4500 7350 0    50   ~ 0
-GND
-Text Label 4500 7450 0    50   ~ 0
+Text Label 3700 7250 0    50   ~ 0
+GND
+Text Label 3700 7350 0    50   ~ 0
 Buck_Out
-Text Label 3850 7350 0    50   ~ 0
-GND
-Text Label 3850 7450 0    50   ~ 0
+Text Label 3300 7300 0    50   ~ 0
+GND
+Text Label 3300 7400 0    50   ~ 0
 Buck_Out
-Text Label 3200 7350 0    50   ~ 0
-GND
-Text Label 3200 7450 0    50   ~ 0
+Text Label 3000 7300 0    50   ~ 0
+GND
+Text Label 3000 7400 0    50   ~ 0
 Buck_Out
 Wire Wire Line
-	8250 5550 8550 5550
-Wire Wire Line
-	8250 5350 8550 5350
+	8250 5250 8550 5250
+Wire Wire Line
+	8250 5150 8550 5150
 Connection ~ 9950 5750
 $Comp
@@
 Wire Wire Line
 	4150 1200 4750 1200
+$Comp
+L Connector:Conn_01x02_Male J18
+U 1 1 60BDCC2D
+P 2850 6900
+F 0 "J18" H 2956 7078 50  0000 C CNN
+F 1 "Battery_out" H 2956 6987 50  0000 C CNN
+F 2 "footprint:input" H 2850 6900 50  0001 C CNN
+F 3 "~" H 2850 6900 50  0001 C CNN
+	1    2850 6900
+	1    0    0    -1
+$EndComp
+Text Label 3050 6900 0    50   ~ 0
+RV1
+Text Label 3050 7000 0    50   ~ 0
+GND
+$Comp
+L Connector:Conn_01x02_Male J19
+U 1 1 60BF90E1
+P 3700 6900
+F 0 "J19" H 3806 7078 50  0000 C CNN
+F 1 "Battery_out" H 3806 6987 50  0000 C CNN
+F 2 "footprint:input" H 3700 6900 50  0001 C CNN
+F 3 "~" H 3700 6900 50  0001 C CNN
+	1    3700 6900
+	1    0    0    -1
+$EndComp
+Text Label 3900 6900 0    50   ~ 0
+RV1
+Text Label 3900 7000 0    50   ~ 0
+GND
+$Comp
+L Connector:Conn_01x02_Male J20
+U 1 1 60C0732F
+P 4100 6900
+F 0 "J20" H 4206 7078 50  0000 C CNN
+F 1 "Battery_out" H 4206 6987 50  0000 C CNN
+F 2 "footprint:input" H 4100 6900 50  0001 C CNN
+F 3 "~" H 4100 6900 50  0001 C CNN
+	1    4100 6900
+	1    0    0    -1
+$EndComp
+Text Label 4300 6900 0    50   ~ 0
+RV1
+Text Label 4300 7000 0    50   ~ 0
+GND
+$Comp
+L Connector:Conn_01x02_Male J21
+U 1 1 60C15580
+P 4400 6900
+F 0 "J21" H 4506 7078 50  0000 C CNN
+F 1 "Battery_out" H 4506 6987 50  0000 C CNN
+F 2 "footprint:input" H 4400 6900 50  0001 C CNN
+F 3 "~" H 4400 6900 50  0001 C CNN
+	1    4400 6900
+	1    0    0    -1
+$EndComp
+Text Label 4600 6900 0    50   ~ 0
+RV1
+Text Label 4600 7000 0    50   ~ 0
+GND
+$Comp
+L Connector:Conn_01x02_Male J22
+U 1 1 60C15810
+P 10350 6750
+F 0 "J22" H 10456 6928 50  0000 C CNN
+F 1 "Conn_01x02_Male" H 10456 6837 50  0000 C CNN
+F 2 "footprint:01x02" H 10350 6750 50  0001 C CNN
+F 3 "~" H 10350 6750 50  0001 C CNN
+	1    10350 6750
+	1    0    0    -1
+$EndComp
+Text Label 10250 6150 0    50   ~ 0
+TX
+Text Label 10250 6050 0    50   ~ 0
+RX
+Wire Wire Line
+	10250 6050 9950 6050
+Wire Wire Line
+	10250 6150 9950 6150
+Text Label 10850 6850 0    50   ~ 0
+TX
+Text Label 10850 6750 0    50   ~ 0
+RX
+Wire Wire Line
+	10850 6750 10550 6750
+Wire Wire Line
+	10850 6850 10550 6850
+Connection ~ 8550 6150
+Wire Wire Line
+	8550 6150 8600 6150
 $EndSCHEMATC

Commit message: issue resolved
Parts:
- added H1, H2, H3, H4: MountingHole, MountingHole:MountingHole_3.2mm_M3, symbol Mechanical:MountingHole
- Q1, Q3: symbol SIS427EDN-T1-GE3:SIS427EDN-T1-GE3 -> PowerBoard-rescue:SIS427EDN-T1-GE3-SIS427EDN-T1-GE3
Changed lines of the file:
@@
 $EndComp
-Wire Wire Line
-	2600 -350 2600 -300
 Wire Wire Line
 	2300 1650 2150 1650
@@
 	4750 1600 4750 1650
 $Comp
-L SIS427EDN-T1-GE3:SIS427EDN-T1-GE3 Q1
+L PowerBoard-rescue:SIS427EDN-T1-GE3-SIS427EDN-T1-GE3 Q1
 U 1 1 60BBC978
 P 2550 800
@@
 Hard kill\n
 $Comp
-L SIS427EDN-T1-GE3:SIS427EDN-T1-GE3 Q3
+L PowerBoard-rescue:SIS427EDN-T1-GE3-SIS427EDN-T1-GE3 Q3
 U 1 1 60C7A442
 P 5150 800
@@
 Wire Wire Line
 	8550 6150 8600 6150
+$Comp
+L Mechanical:MountingHole H2
+U 1 1 60BF09A7
+P 6500 4300
+F 0 "H2" H 6600 4346 50  0000 L CNN
+F 1 "MountingHole" H 6600 4255 50  0000 L CNN
+F 2 "MountingHole:MountingHole_3.2mm_M3" H 6500 4300 50  0001 C CNN
+F 3 "~" H 6500 4300 50  0001 C CNN
+	1    6500 4300
+	1    0    0    -1
+$EndComp
+$Comp
+L Mechanical:MountingHole H3
+U 1 1 60BF0BC4
+P 6500 4500
+F 0 "H3" H 6600 4546 50  0000 L CNN
+F 1 "MountingHole" H 6600 4455 50  0000 L CNN
+F 2 "MountingHole:MountingHole_3.2mm_M3" H 6500 4500 50  0001 C CNN
+F 3 "~" H 6500 4500 50  0001 C CNN
+	1    6500 4500
+	1    0    0    -1
+$EndComp
+$Comp
+L Mechanical:MountingHole H4
+U 1 1 60BFF79A
+P 6500 4700
+F 0 "H4" H 6600 4746 50  0000 L CNN
+F 1 "MountingHole" H 6600 4655 50  0000 L CNN
+F 2 "MountingHole:MountingHole_3.2mm_M3" H 6500 4700 50  0001 C CNN
+F 3 "~" H 6500 4700 50  0001 C CNN
+	1    6500 4700
+	1    0    0    -1
+$EndComp
+$Comp
+L Mechanical:MountingHole H1
+U 1 1 60C0E33B
+P 6500 4100
+F 0 "H1" H 6600 4146 50  0000 L CNN
+F 1 "MountingHole" H 6600 4055 50  0000 L CNN
+F 2 "MountingHole:MountingHole_3.2mm_M3" H 6500 4100 50  0001 C CNN
+F 3 "~" H 6500 4100 50  0001 C CNN
+	1    6500 4100
+	1    0    0    -1
+$EndComp
 $EndSCHEMATC
