File: ESC-board/4ESC_board/4ESC_board.sch (KiCad schematic (older format))
At the start: 9 parts, among them U1 ESCPINS, U2 ESCPINS, U3 ESCPINS, U4 ESCPINS

Commit message: PCBlayout, Routing, 3DModels, DONE
Parts:
- C1: footprint (none) -> molex:molex_supersabre_1x2_172043-0201
- C3: footprint (none) -> molex:Molex_microfit_2x6_444281201
Connections:
- net TB1: now also C3.6; no longer C3.12
- net TB2: now also C3.10; no longer C3.6
- net TB3: now also C3.7; no longer C3.3
- net TB4: now also C3.3; no longer C3.9
- net TG1: now also C3.5; no longer C3.11
- net TG2: now also C3.11; no longer C3.5
- net TG3: now also C3.8; no longer C3.2
- net TG4: now also C3.2; no longer C3.8
- net TW1: now also C3.4; no longer C3.10
- net TW2: now also C3.12; no longer C3.4
- net TW3: now also C3.9; no longer C3.1
- net TW4: now also C3.1; no longer C3.7
Changed lines of the file:
@@
 U 1 1 5FEA0F57
 P 6250 4300
-F 0 "C3" H 5912 4254 50  0000 R CNN
+F 0 "C3" H 5912 4254 50  0000 C CNN
 F 1 "6x2_connector" H 5912 4345 50  0000 R CNN
-F 2 "" H 6250 4300 50  0001 C CNN
+F 2 "molex:Molex_microfit_2x6_444281201" H 6250 4300 50  0001 C CNN
 F 3 "" H 6250 4300 50  0001 C CNN
 	1    6250 4300
-	-1   0    0    1
+	-1   0    0    -1
 $EndComp
 $Comp
@@
 F 0 "C1" V 1399 1528 50  0000 L CNN
 F 1 "1x2_connector" V 1490 1528 50  0000 L CNN
-F 2 "" H 1750 1250 50  0001 C CNN
+F 2 "molex:molex_supersabre_1x2_172043-0201" H 1750 1250 50  0001 C CNN
 F 3 "" H 1750 1250 50  0001 C CNN
 	1    1450 1450
@@
 Text Label 6200 4500 3    50   ~ 0
 TW1
-Text Label 6000 4100 1    50   ~ 0
+Text Label 6200 4100 1    50   ~ 0
 TB2
 Text Label 6100 4100 1    50   ~ 0
 TG2
-Text Label 6200 4100 1    50   ~ 0
+Text Label 6000 4100 1    50   ~ 0
 TW2
-Text Label 6300 4100 1    50   ~ 0
+Text Label 6500 4100 1    50   ~ 0
 TB3
 Text Label 6400 4100 1    50   ~ 0
 TG3
-Text Label 6500 4100 1    50   ~ 0
+Text Label 6300 4100 1    50   ~ 0
 TW3
 Text Label 6400 4500 3    50   ~ 0

Commit message: added fuse
Parts:
- added F1: Fuse, minibladefuse:MCCQ-122, symbol Device:Fuse
Connections:
- net GND: now also F1.1; no longer C1.2
- new net: C1.2, F1.2
Changed lines of the file:
@@
 Text Label 1250 1400 2    50   ~ 0
 VIN
-Text Label 1250 1500 2    50   ~ 0
+Text Label 1250 1800 3    50   ~ 0
 GND
 Text Label 6000 4500 3    50   ~ 0
@@
 Text Label 2750 950  0    50   ~ 0
 GND
+$Comp
+L Device:Fuse F1
+U 1 1 6232DC6A
+P 1250 1650
+F 0 "F1" V 1350 1650 50  0000 C CNN
+F 1 "Fuse" V 1144 1650 50  0000 C CNN
+F 2 "minibladefuse:MCCQ-122" V 1180 1650 50  0001 C CNN
+F 3 "" H 1250 1650 50  0001 C CNN
+	1    1250 1650
+	-1   0    0    1
+$EndComp
 $EndSCHEMATC
